File: lora_module.kicad_sch (KiCad schematic)
At the start: 0 parts

Commit message: feat(lora): Add LoRa module to schematic
This commit adds the LoRa module and its associated components to the
`lora_module.kicad_sch` schematic sheet.

- Added the LoRa module symbol (Ai-Thinker-Ra-02).
Parts:
- added U1: Ai-Thinker-Ra-02, RF_Module:Ai-Thinker-Ra-01-LoRa, symbol RF_Module:Ai-Thinker-Ra-02
Connections:
- new net: U1.1 (GND), U1.16 (GND), U1.2 (GND), U1.9 (GND)
Changed lines of the file:
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@@
 	(generator_version "9.0")
 	(paper "A4")
+	(symbol
+		(lib_id "RF_Module:Ai-Thinker-Ra-02")
+		(at 146.05 102.87 0)
+		(unit 1)
+		(exclude_from_sim no)
+		(in_bom yes)
+		(on_board yes)
+		(dnp no)
+		(fields_autoplaced yes)
+		(property "Reference" "U1"
+			(at 148.1933 85.09 0)
+			(effects
+				(font
+					(size 1.27 1.27)
+				)
+				(justify left)
+			)
+		)
+		(property "Value" "Ai-Thinker-Ra-02"
+			(at 148.1933 87.63 0)
+			(effects
+				(font
+					(size 1.27 1.27)
+				)
+				(justify left)
+			)
+		)
+		(property "Footprint" "RF_Module:Ai-Thinker-Ra-01-LoRa"
+			(at 171.45 113.03 0)
+			(effects
+				(font
+					(size 1.27 1.27)
+				)
+				(hide yes)
+			)
+		)
+		(property "Datasheet" "http://wiki.ai-thinker.com/_media/lora/docs/c048ps01a1_ra-02_product_specification_v1.1.pdf"
+			(at 148.59 83.82 0)
+			(effects
+				(font
+					(size 1.27 1.27)
+				)
+				(hide yes)
+			)
+		)
+		(property "Description" "Ai-Thinker Ra-02 410-525 MHz LoRa Module, SPI interface, U.FL antenna connector"
+			(at 146.05 102.87 0)
+			(effects
+				(font
+					(size 1.27 1.27)
+				)
+				(hide yes)
+			)
+		)
+		(pin "10"
+		)
+		(pin "5"
+		)
+		(pin "6"
+		)
+		(pin "9"
+		)
+		(pin "4"
+		)
+		(pin "2"
+		)
+		(pin "11"
+		)
+		(pin "1"
+		)
+		(pin "12"
+		)
+		(pin "16"
+		)
+		(pin "8"
+		)
+		(pin "7"
+		)
+		(pin "13"
+		)
+		(pin "14"
+		)
+		(pin "3"
+		)
+		(pin "15"
+		)
+		(instances
+			(project ""
+				(path "/01550cd7-b424-469c-925b-c370f3609cd4/2dab47df-4ca4-4373-b48e-0efc8c61f605"
+					(reference "U1")
+					(unit 1)
+				)
+			)
+		)
+	)
 )
